Commit message: test moveit failed

File: src/robot/urdf/gazebo.xacro (robot description, xacro)
@@ -13,6 +13,12 @@
                 <box size="0.05 0.05 0.05"/>
             </geometry>
-            <material name="black"/>
+            <material name="black">
+                <color rgba="0 0 0 1"/> </material>
         </visual>
+        <collision>
+            <geometry>
+                <box size="0.05 0.05 0.05"/>
+            </geometry>
+        </collision>
     </link>
     <joint name="camera_joint" type="fixed">
@@ -22,5 +28,5 @@
     </joint>
     <gazebo reference="camera_link">
-        <sensor name="camera" type="camera">
+        <material>Gazebo/Black</material> <sensor name="camera" type="camera">
             <camera>
                 <horizontal_fov>1.047</horizontal_fov>
@@ -37,5 +43,6 @@
             <update_rate>30</update_rate>
             <visualize>true</visualize>
-            <topic>camera/image_raw</topic> </sensor>
+            <topic>camera/image_raw</topic>
+        </sensor>
     </gazebo>
 </robot>

File: src/robot/urdf/robot.ros2_control.xacro (robot description, xacro)
@@ -7,24 +7,10 @@
                 <xacro:if value="${use_sim}">
                     <plugin>gz_ros2_control/GazeboSimSystem</plugin>
-                    <parameters>$(find robot_moveit)/config/ros2_controllers.yaml</parameters>
                 </xacro:if>
                 <xacro:unless value="${use_sim}">
                     <plugin>mock_components/GenericSystem</plugin>
+                    <param name="calculate_dynamics">true</param>
                 </xacro:unless>
             </hardware>
-            <joint name="joint_gl">
-                <command_interface name="position"/>
-                <state_interface name="position">
-                  <param name="initial_value">${initial_positions['joint_gl']}</param>
-                </state_interface>
-                <state_interface name="velocity"/>
-            </joint>
-            <joint name="joint_gr">
-                <command_interface name="position"/>
-                <state_interface name="position">
-                  <param name="initial_value">${initial_positions['joint_gr']}</param>
-                </state_interface>
-                <state_interface name="velocity"/>
-            </joint>
             <joint name="joint_1">
                 <command_interface name="position"/>
@@ -69,4 +55,18 @@
                 <state_interface name="velocity"/>
             </joint>
+            <joint name="joint_gl">
+                <command_interface name="position"/>
+                <state_interface name="position">
+                  <param name="initial_value">${initial_positions['joint_gl']}</param>
+                </state_interface>
+                <state_interface name="velocity"/>
+            </joint>
+            <joint name="joint_gr">
+                <command_interface name="position"/>
+                <state_interface name="position">
+                  <param name="initial_value">${initial_positions['joint_gr']}</param>
+                </state_interface>
+                <state_interface name="velocity"/>
+            </joint>
         </ros2_control>
     </xacro:macro>
