Commit message: clearn xacro

File: src/robot_description/urdf/materials.xacro (robot description, xacro)
@@ -1,15 +1,21 @@
 <?xml version="1.0" ?>
-<robot name="panda" xmlns:xacro="http://www.ros.org/wiki/xacro">
-  <material name="red">
-    <color rgba="1.0 0.0 0.0 1.000"/>
+<robot name ="panda" xmlns:xacro="http://www.ros.org/wiki/xacro">
+  <material name  ="black">
+    <color  rgba  ="0.0 0.0 0.0 1.0"/>
   </material>
-  <material name="green">
-    <color rgba="0.0 1.0 0.0 1.000"/>
+  <material name  ="white">
+    <color  rgba  ="1.0 1.0 1.0 1.0"/>
   </material>
-  <material name="blue">
-    <color rgba="0.0 0.0 1.0 1.000"/>
+  <material name  ="red">
+    <color  rgba  ="0.8 0.0 0.0 1.0"/>
   </material>
-  <material name="black">
-    <color rgba="1.0 1.0 1.0 1.000"/>
+  <material name  ="blue">
+    <color  rgba  ="0.0 0.0 0.8 1.0"/>
+  </material>
+  <material name  ="green">
+    <color  rgba  ="0.0 0.8 0.0 1.0"/>
+  </material>
+  <material name  ="grey">
+    <color  rgba  ="0.5 0.5 0.5 1.0"/>
   </material>
 </robot>

File: src/robot_description/urdf/robot.urdf.xacro (robot description, xacro)
@@ -1,6 +1,8 @@
 <?xml version="1.0"?>
-<robot xmlns:xacro="http://www.ros.org/wiki/xacro" name="robot">
-    <xacro:arg name="use_sim" default="true" />
-    <xacro:arg name="initial_positions_file" default="$(find robot_moveit)/config/initial_positions.yaml" />
+<robot xmlns:xacro ="http://www.ros.org/wiki/xacro" name="robot">
+    <xacro:arg name ="use_sim"
+            default ="true" />
+    <xacro:arg name ="initial_positions_file"
+            default ="$(find robot_moveit)/config/initial_positions.yaml" />
     <xacro:include filename =   "$(find robot_description)/urdf/materials.xacro" />
     <xacro:include filename =   "$(find robot_description)/urdf/robot.xacro" />
@@ -8,6 +10,11 @@
     <xacro:include filename =   "$(find robot_description)/urdf/robot.ros2_control.xacro" />
     <xacro:include filename =   "$(find robot_description)/urdf/gazebo.xacro" />
-    <xacro:base_camera parent_link  = "base_link"/>
-    <xacro:robot_ros2_control name  ="robot"
+    <xacro:base_camera
+            parent_link             ="base_link"
+            base_link               ="astra_link"
+            camera_name             ="astra_depth"
+            frame_name              ="astra_link"/>
+    <xacro:robot_ros2_control
+            name                    ="robot"
             initial_positions_file  ="$(arg initial_positions_file)"
             use_sim                 ="$(arg use_sim)" />

File: src/robot_description/urdf/robot.xacro (robot description, xacro)
@@ -1,333 +1,344 @@
 <?xml version="1.0"?>
 <robot name="robot" xmlns:xacro="http://www.ros.org/wiki/xacro">
+  <!-- ________________ DEFINE LINK ________________________________________________________________________ -->
   <!-- World Frame -->
-  <link name="world"/>
- <!-- World-Base Joint -->
-  <joint name="virtual_joint" type="fixed">
-      <parent link="world"/>
-      <child link="base_link"/>
-      <origin xyz="0 0 0" rpy="0 0 0"/>
-  </joint>
+  <link name  ="world"/>
+  <link name  ="tcp_link"/>
   <!-- Link 0 - Base -->
-  <link name="base_link">
-    <inertial>
-      <origin xyz="-0.00544954615598158 0.000157418519134474 0.00564099250157026" rpy="0 0 0" />
-      <mass value="1.78696933370067" />
-      <inertia
-        ixx="0.00334289861376234"   ixy="-2.39019225970563E-07"
-        ixz="7.11788112309683E-06"  iyy="0.0031863560397784"
-        iyz="-2.78684112590384E-06" izz="0.00645191220467659" />
+  <link name  ="base_link">
+    <inertial>
+      <origin xyz ="-0.00544954615598158 0.000157418519134474 0.00564099250157026" rpy="0 0 0" />
+      <mass value ="1.78696933370067" />
+      <inertia
+              ixx ="0.00334289861376234"
+              ixy ="-2.39019225970563E-07"
+              ixz ="7.11788112309683E-06"
+              iyy ="0.0031863560397784"
+              iyz ="-2.78684112590384E-06"
+              izz ="0.00645191220467659" />
+    </inertial>
+    <visual>
+      <origin xyz ="0 0 0" rpy  ="0 0 0" />
+      <geometry>
+        <mesh filename  ="package://robot_description/meshes/base_link.stl" />
+      </geometry>
+      <material   name  ="white"></material>
+    </visual>
+    <collision>
+      <origin xyz ="0 0 0" rpy ="0 0 0" />
+      <geometry>
+        <mesh filename  ="package://robot_description/meshes/base_link.stl" />
+      </geometry>
+    </collision>
+  </link>
+  <!-- Link 1 -->
+  <link name  ="link_1">
+    <inertial>
+      <origin   xyz  ="0.0193443558112907 0.0109921802765565 0.0924758072620357" rpy="0 0 0" />
+      <mass   value  ="5.50396042361908" />
+      <inertia
+                ixx ="0.0130037829993516"
+                ixy ="3.49214734799824E-09"
+                ixz ="-0.00313572650782407"
+                iyy ="0.0174211851360363"
+                iyz ="-2.33013746145458E-06"
+                izz ="0.0140359346087906" />
+    </inertial>
+    <visual>
+      <origin xyz ="0 0 0" rpy  ="0 0 0" />
+      <geometry>
+        <mesh filename  ="package://robot_description/meshes/link_1.stl" />
+      </geometry>
+      <material   name  ="white"></material>
+    </visual>
+    <collision>
+      <origin xyz ="0 0 0" rpy  ="0 0 0" />
+      <geometry>
+        <mesh filename  ="package://robot_description/meshes/link_1.stl" />
+      </geometry>
+    </collision>
+  </link>
+    <!-- Link 2 -->
+  <link name="link_2">
+    <inertial>
+      <origin xyz ="0.095965941991434 0.000112006139674839 -0.0319594915411429"  rpy="0 0 0" />
+      <mass value ="2.68614147040981" />
+      <inertia
+              ixx ="0.00216208190226954"
+              ixy ="7.03906699411074E-07"
+              ixz ="1.9470092472916E-06"
+              iyy ="0.0110452906557092"
+              iyz ="-1.43932327786374E-06"
+              izz ="0.0125902837214324" />
     </inertial>
     <visual>
       <origin xyz="0 0 0" rpy="0 0 0" />
       <geometry>
-        <mesh filename="package://robot_description/meshes/base_link.stl" />
-      </geometry>
-      <material name="">
-        <color rgba="0.752941176470588 0.752941176470588 0.752941176470588 1" />
-      </material>
+        <mesh   filename ="package://robot_description/meshes/link_2.stl" />
+      </geometry>
+      <material     name  ="white"></material>
     </visual>
     <collision>
       <origin xyz="0 0 0" rpy="0 0 0" />
       <geometry>
-        <mesh filename="package://robot_description/meshes/base_link.stl" />
-      </geometry>
-    </collision>
-  </link>
-    <!-- Link 1 -->
-  <link name="link_1">
-    <inertial>
-      <origin xyz="0.0193443558112907 0.0109921802765565 0.0924758072620357" rpy="0 0 0" />
-      <mass  value="5.50396042361908" />
-      <inertia
-        ixx="0.0130037829993516"    ixy="3.49214734799824E-09"
-        ixz="-0.00313572650782407"  iyy="0.0174211851360363"
-        iyz="-2.33013746145458E-06" izz="0.0140359346087906" />
+        <mesh filename="package://robot_description/meshes/link_2.stl" />
+      </geometry>
+    </collision>
+  </link>
+    <!-- Link 3 -->
+  <link  name="link_3">
+    <inertial>
+      <origin xyz ="0.0315400667409967 -0.0522316930638639 -0.0372996788949479" rpy="0 0 0" />
+      <mass value ="2.69379315969066" />
+      <inertia
+              ixx ="0.00297065150537785"
+              ixy ="0.000173737882412212"
+              ixz ="1.08004336423003E-07"
+              iyy ="0.0019143128411473"
+              iyz ="4.2036787275891E-06"
+              izz ="0.0039181139326064" />
+    </inertial>
+    <visual>
+      <origin  xyz="0 0 0" rpy="0 0 0" />
+      <geometry>
+        <mesh  filename="package://robot_description/meshes/link_3.stl" />
+      </geometry>
+      <material name="white"></material>
+    </visual>
+    <collision>
+      <origin  xyz="0 0 0" rpy="0 0 0" />
+      <geometry>
+        <mesh  filename="package://robot_description/meshes/link_3.stl" />
+      </geometry>
+    </collision>
+  </link>
+    <!-- Link 4 -->
+  <link  name="link_4">
+    <inertial>
+      <origin xyz ="0.00868566509472264 -0.000351062944789704 0.0358084533663054" rpy="0 0 0" />
+      <mass value ="1.80796623919651" />
+      <inertia
+              ixx ="0.00163140667717977"
+              ixy ="-1.5364988555156E-06"
+              ixz ="-1.21111109518308E-05"
+              iyy ="0.00126669781876782"
+              iyz ="-8.97475562349671E-07"
+              izz ="0.0010711724867268" />
+    </inertial>
+    <visual>
+      <origin xyz="0 0 0"  rpy="0 0 0" />
+      <geometry>
+        <mesh filename="package://robot_description/meshes/link_4.stl" />
+      </geometry>
+      <material name="white"></material>
+    </visual>
+    <collision>
+      <origin  xyz="0 0 0"  rpy="0 0 0" />
+      <geometry>
+        <mesh filename="package://robot_description/meshes/link_4.stl" />
+      </geometry>
+    </collision>
+  </link>
+    <!-- Link 5 -->
+  <link  name="link_5">
+    <inertial>
+      <origin xyz ="0.0674634334441427 5.73631023903509E-05 0.00771105147453628" rpy="0 0 0" />
+      <mass value ="0.367372399298886" />
+      <inertia
+              ixx ="0.000203467788892474"
+              ixy ="-4.31988988741858E-07"
+              ixz ="-2.92876701433074E-05"
+              iyy ="0.000404007801086554"
+              iyz ="-9.06114097030996E-09"
+              izz ="0.000453819777422173" />
     </inertial>
     <visual>
       <origin xyz="0 0 0" rpy="0 0 0" />
       <geometry>
-        <mesh filename="package://robot_description/meshes/link_1.stl" />
-      </geometry>
-      <material name="">
-        <color rgba="0.752941176470588 0.752941176470588 0.752941176470588 1" />
-      </material>
-    </visual>
-    <collision>
-      <origin xyz="0 0 0" rpy="0 0 0" />
-      <geometry>
-        <mesh filename="package://robot_description/meshes/link_1.stl" />
-      </geometry>
-    </collision>
-  </link>
-    <!--................. JOINT 1..................................-->
-  <joint name="joint_1" type="revolute">
-    <origin xyz="0 0 0.01" rpy="0 0 0" />
-    <parent link="base_link" />
-    <child link="link_1" />
-    <axis xyz="0 0 1" />
-    <limit
-      lower="-2.0943" upper="2.0943"
-      effort="1000" velocity="5.0" />
-  </joint>
-  <!-- Link 2 -->
-  <link name="link_2">
-    <inertial>
-      <origin
-        xyz="0.095965941991434 0.000112006139674839 -0.0319594915411429"  rpy="0 0 0" />
-      <mass value="2.68614147040981" />
-      <inertia
-        ixx="0.00216208190226954" ixy="7.03906699411074E-07"
-        ixz="1.9470092472916E-06" iyy="0.0110452906557092"
-        iyz="-1.43932327786374E-06" izz="0.0125902837214324" />
-    </inertial>
-    <visual>
-      <origin xyz="0 0 0" rpy="0 0 0" />
-      <geometry>
-        <mesh  filename="package://robot_description/meshes/link_2.stl" />
-      </geometry>
-      <material name="">
-        <color  rgba="0.752941176470588 0.752941176470588 0.752941176470588 1" />
-      </material>
-    </visual>
-    <collision>
-      <origin xyz="0 0 0" rpy="0 0 0" />
-      <geometry>
-        <mesh filename="package://robot_description/meshes/link_2.stl" />
-      </geometry>
-    </collision>
-  </link>
-    <!--................. JOINT 2..................................-->
-  <joint  name="joint_2" type="revolute">
-     <origin  xyz="0.1 0.05 0.24313"  rpy="-1.5707963267949 -1.5707963267949 0" />
-    <parent link="link_1" />
-    <child link="link_2" />
-    <axis  xyz="0 0 1" />
-    <limit
-      lower="-1.5707" upper="2.6179"
-      effort="1000" velocity="5.0" />
-  </joint>
-  <!-- Link 3 -->
-  <link  name="link_3">
-    <inertial>
-      <origin
-        xyz="0.0315400667409967 -0.0522316930638639 -0.0372996788949479"
-        rpy="0 0 0" />
-      <mass value="2.69379315969066" />
-      <inertia
-        ixx="0.00297065150537785" ixy="0.000173737882412212"
-        ixz="1.08004336423003E-07" iyy="0.0019143128411473"
-        iyz="4.2036787275891E-06" izz="0.0039181139326064" />
-    </inertial>
-    <visual>
-      <origin  xyz="0 0 0" rpy="0 0 0" />
-      <geometry>
-        <mesh  filename="package://robot_description/meshes/link_3.stl" />
-      </geometry>
-      <material name="">
-        <color rgba="0.752941176470588 0.752941176470588 0.752941176470588 1" />
-      </material>
-    </visual>
-    <collision>
-      <origin  xyz="0 0 0" rpy="0 0 0" />
-      <geometry>
-        <mesh  filename="package://robot_description/meshes/link_3.stl" />
-      </geometry>
-    </collision>
-  </link>
-    <!--................. JOINT 3..................................-->
-  <joint  name="joint_3" type="revolute">
-    <origin  xyz="0.25 0 -0.01"  rpy="0 0 1.57079632679489" />
-    <parent link="link_2" />
-    <child link="link_3" />
-    <axis  xyz="0 0 1" />
-    <limit
-      lower="-1.5707" upper="1.5707"
-      effort="1000"  velocity="5.0" />
-  </joint>
-  <!-- Link 4 -->
-  <link  name="link_4">
-    <inertial>
-      <origin xyz="0.00868566509472264 -0.000351062944789704 0.0358084533663054" rpy="0 0 0" />
-      <mass value="1.80796623919651" />
-      <inertia
-        ixx="0.00163140667717977"   ixy="-1.5364988555156E-06"
-        ixz="-1.21111109518308E-05" iyy="0.00126669781876782"
-        iyz="-8.97475562349671E-07" izz="0.0010711724867268" />
-    </inertial>
-    <visual>
-      <origin xyz="0 0 0"  rpy="0 0 0" />
-      <geometry>
-        <mesh filename="package://robot_description/meshes/link_4.stl" />
-      </geometry>
-      <material  name="">
-        <color rgba="0.752941176470588 0.752941176470588 0.752941176470588 1" />
-      </material>
+        <mesh filename  ="package://robot_description/meshes/link_5.stl" />
+      </geometry>
+      <material   name  ="white"></material>
     </visual>
     <collision>
       <origin  xyz="0 0 0"  rpy="0 0 0" />
       <geometry>
-        <mesh filename="package://robot_description/meshes/link_4.stl" />
-      </geometry>
-    </collision>
-  </link>
-   <!--................. JOINT 4..................................-->
-  <joint  name="joint_4" type="revolute">
-    <origin  xyz="0.103 -0.09 -0.04"  rpy="0 1.5708 0" />
-    <parent   link="link_3" />
-    <child  link="link_4" />
-    <axis xyz="0 0 1" />
-    <limit
-      lower="-1.5707" upper="1.5707"
-      effort="1000" velocity="5.0" />
-  </joint>
-  <!-- Link 5 -->
-  <link  name="link_5">
-    <inertial>
-      <origin xyz="0.0674634334441427 5.73631023903509E-05 0.00771105147453628" rpy="0 0 0" />
-      <mass   value="0.367372399298886" />
-      <inertia
-        ixx="0.000203467788892474"   ixy="-4.31988988741858E-07"
-        ixz="-2.92876701433074E-05"  iyy="0.000404007801086554"
-        iyz="-9.06114097030996E-09"  izz="0.000453819777422173" />
-    </inertial>
-    <visual>
-      <origin xyz="0 0 0" rpy="0 0 0" />
-      <geometry>
-        <mesh filename="package://robot_description/meshes/link_5.stl" />
-      </geometry>
-      <material name="">
-        <color rgba="0.752941176470588 0.752941176470588 0.752941176470588 1" />
-      </material>
-    </visual>
-    <collision>
-      <origin  xyz="0 0 0"  rpy="0 0 0" />
-      <geometry>
-        <mesh filename="package://robot_description/meshes/link_5.stl" />
-      </geometry>
-    </collision>
-  </link>
-    <!--................. JOINT 5..................................-->
-  <joint name="joint_5" type="revolute">
-    <origin  xyz="-0.0134 0 0.12"  rpy="3.1416 -1.5708 3.1416" />
-    <parent link="link_4" />
-    <child link="link_5" />
-    <axis xyz="0 0 1" />
-    <limit
-      lower="-1.5707" upper="1.5707"
-      effort="1000" velocity="5.0" />
-  </joint>
-  <!-- Link 6 -->
+        <mesh filename  ="package://robot_description/meshes/link_5.stl" />
+      </geometry>
+    </collision>
+  </link>
+    <!-- Link 6 -->
   <link  name="link_6">
     <inertial>
-      <origin xyz="-3.2560015697054E-06 -3.69429945190625E-07 -0.000227999228200271" rpy="0 0 0" />
-      <mass value="0.0760881236172958" />
-      <inertia
-        ixx="1.0689375645495E-05"   ixy="1.29742190426518E-07"
-        ixz="-4.13087402822219E-09" iyy="6.01775641263719E-05"
-        iyz="-8.47409888919864E-11" izz="6.20472722814015E-05" />
-    </inertial>
-    <visual>
-      <origin xyz="0 0 0" rpy="0 0 0" />
-      <geometry>
-        <mesh filename="package://robot_description/meshes/link_6.stl" />
-      </geometry>
-      <material name="">
-        <color rgba="0.752941176470588 0.752941176470588 0.752941176470588 1" />
-      </material>
-    </visual>
-    <collision>
-      <origin  xyz="0 0 0"  rpy="0 0 0" />
-      <geometry>
-        <mesh
-          filename="package://robot_description/meshes/link_6.stl" />
-      </geometry>
-    </collision>
-  </link>
-<!--................. JOINT 6..................................-->
-  <joint name="joint_6"  type="revolute">
-    <origin  xyz="0.136 0 -0.0148299999999991"  rpy="0 -1.5708 3.1415" />
-    <parent link="link_5" />
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
File: src/robot_description/urdf/sensors.xacro (robot description, xacro)
@@ -1,10 +1,14 @@
 <?xml version="1.0"?>
 <robot xmlns:xacro="http://www.ros.org/wiki/xacro">
-  <xacro:macro  name="base_camera" params="parent_link base_link:=camera_link">
-    <link       name="${base_link}">
+  <xacro:macro  name  ="base_camera"
+              params  ="parent_link
+                        base_link     := camera_link
+                        camera_name   := camera
+                        frame_name    := frame">
+    <link       name  ="${base_link}">
       <inertial>
-        <origin   xyz   ="0 0 0" rpy  ="0 0 0"/>
-        <mass     value ="0.1"/>
-        <inertia  ixx   ="0.1"   ixy  ="0" ixz="0" iyy="0.1" iyz="0" izz="0.1"/>
+        <origin xyz   ="0 0 0" rpy  ="0 0 0"/>
+        <mass   value ="0.1"/>
+        <inertia  ixx ="0.1"   ixy  ="0" ixz="0" iyy="0.1" iyz="0" izz="0.1"/>
       </inertial>
       <visual>
@@ -20,25 +24,21 @@
       </collision>
     </link>
-    <link         name  ="${base_link}_optical"/>
+    <link           name  ="${base_link}_optical"/>
     <!-- chỉnh lại pose camera tại đây -->
-    <joint        name  ="${base_link}_joint" type="fixed">
-      <parent     link  ="${parent_link}"/>
-      <child      link  ="${base_link}"/>
-      <origin     xyz   ="0.6 0 1.0" rpy="3.1415 0 1.5707"/>
+    <joint          name  ="${base_link}_joint"         type  ="fixed">
+      <parent       link  ="${parent_link}"/>
+      <child        link  ="${base_link}"/>
+      <origin       xyz   ="0.6 0 1.0" rpy="${pi} 0 ${pi/2}"/>
     </joint>
     <!-- Chỉnh lại optical frame -->
-    <joint        name  ="${base_link}_optical_joint" type="fixed">
-      <parent     link  ="${base_link}"/>
-      <child      link  ="${base_link}_optical"/>
-      <origin     xyz   ="0 0 0" rpy="0 0 0"/>
+    <joint          name  ="${base_link}_optical_joint" type  ="fixed">
+      <parent       link  ="${base_link}"/>
+      <child        link  ="${base_link}_optical"/>
+      <origin       xyz   ="0 0 0" rpy="0 0 0"/>
     </joint>
-    <gazebo reference="${base_link}">
+    <!--gazebo reference="camera_link">
       <sensor name="camera" type="camera">
-        <pose>0 0 0 0 0 0</pose>
-        <visualize>true</visualize>
-        <always_on>true</always_on>
-        <update_rate>30</update_rate>
-        <camera name="Astra_camera">
-          <horizontal_fov>1.0</horizontal_fov>
+        <camera>
+          <horizontal_fov>1.3962634</horizontal_fov>
           <image>
             <width>640</width>
@@ -47,10 +47,21 @@
           </image>
           <clip>
-            <near>0.05</near>
-            <far>8.0</far>
+            <near>0.1</near>
+            <far>15</far>
           </clip>
+          <noise>
+            <type>gaussian</type>
+            <mean>0.0</mean>
+            <stddev>0.007</stddev>
+          </noise>
+          <optical_frame_id>camera_link_optical</optical_frame_id>
+          <camera_info_topic>camera/camera_info</camera_info_topic>
         </camera>
+        <always_on>1</always_on>
+        <update_rate>20</update_rate>
+        <visualize>true</visualize>
+        <topic>camera/image</topic>
       </sensor>
-    </gazebo>
+    </gazebo-->
   </xacro:macro>
 </robot>
