Commit message: update robot_description_moveit

File: src/robot_description/urdf/gazebo.xacro (robot description, xacro)
@@ -3,6 +3,6 @@
     <xacro:if value="$(arg use_sim)">
         <gazebo>
-            <plugin filename="gz_ros2_control-system" name="gz_ros2_control::GazeboSimROS2ControlPlugin">
-                <parameters>$(find robot_moveit)/config/ros2_controllers.yaml</parameters>
+            <plugin filename="libgz_ros2_control-system.so" name="gz_ros2_control::GazeboSimROS2ControlPlugin">
+            <parameters>$(find robot_description_moveit)/config/ros2_controllers.yaml</parameters>
             </plugin>
         </gazebo>
@@ -14,35 +14,17 @@
             </geometry>
             <material name="black">
-                <color rgba="0 0 0 1"/> </material>
+                <color rgba="0 0 0 1"/>
+            </material>
         </visual>
         <collision>
             <geometry>
-                <box size="0.05 0.05 0.05"/>
+                 <box size="0.05 0.05 0.05"/>
             </geometry>
         </collision>
     </link>
     <joint name="camera_joint" type="fixed">
-        <parent link="world"/>
+        <parent link="base_link"/>
         <child link="camera_link"/>
-        <origin xyz="0.5 0.0 1.5" rpy="0 1.57 0"/>
+        <origin xyz="0.5 0 0.5" rpy="0 0 0"/>
     </joint>
-    <gazebo reference="camera_link">
-        <material>Gazebo/Black</material> <sensor name="camera" type="camera">
-            <camera>
-                <horizontal_fov>1.047</horizontal_fov>
-                <image>
-                    <width>640</width>
-                    <height>480</height>
-                </image>
-                <clip>
-                    <near>0.1</near>
-                    <far>100</far>
-                </clip>
-            </camera>
-            <always_on>1</always_on>
-            <update_rate>30</update_rate>
-            <visualize>true</visualize>
-            <topic>camera/image_raw</topic>
-        </sensor>
-    </gazebo>
 </robot>

File: src/robot_description/urdf/robot.ros2_control.xacro (robot description, xacro)
@@ -26,4 +26,5 @@
         <command_interface name="position"/>
         <state_interface name="position"/>
+        <command_interface name="velocity"/>
         <state_interface name="velocity"/>
       </joint>
@@ -31,4 +32,5 @@
         <command_interface name="position"/>
         <state_interface name="position"/>
+        <command_interface name="velocity"/>
         <state_interface name="velocity"/>
       </joint>
@@ -36,4 +38,5 @@
         <command_interface name="position"/>
         <state_interface name="position"/>
+        <command_interface name="velocity"/>
         <state_interface name="velocity"/>
       </joint>
@@ -41,4 +44,5 @@
         <command_interface name="position"/>
         <state_interface name="position"/>
+        <command_interface name="velocity"/>
         <state_interface name="velocity"/>
       </joint>
@@ -46,4 +50,5 @@
         <command_interface name="position"/>
         <state_interface name="position"/>
+        <command_interface name="velocity"/>
         <state_interface name="velocity"/>
       </joint>
@@ -51,4 +56,5 @@
         <command_interface name="position"/>
         <state_interface name="position"/>
+        <command_interface name="velocity"/>
         <state_interface name="velocity"/>
       </joint>
@@ -56,4 +62,5 @@
         <command_interface name="position"/>
         <state_interface name="position"/>
+        <command_interface name="velocity"/>
         <state_interface name="velocity"/>
       </joint>
@@ -61,4 +68,5 @@
         <command_interface name="position"/>
         <state_interface name="position"/>
+        <command_interface name="velocity"/>
         <state_interface name="velocity"/>
       </joint>

File: src/robot_description/urdf/robot.urdf.xacro (robot description, xacro)
@@ -2,8 +2,8 @@
 <robot xmlns:xacro="http://www.ros.org/wiki/xacro" name="robot">
     <xacro:arg name="use_sim" default="false" />
-   <!--<xacro:arg name="initial_positions_file" default="$(find robot_moveit)/config/initial_positions.yaml" /> -->
+    <xacro:arg name="initial_positions_file" default="$(find robot_description_moveit)/config/initial_positions.yaml" />
     <xacro:include filename="$(find robot_description)/urdf/robot.xacro" />
     <xacro:include filename="$(find robot_description)/urdf/robot.ros2_control.xacro" />
     <xacro:include filename="$(find robot_description)/urdf/gazebo.xacro" />
-    <xacro:robot_ros2_control name="robot_description" initial_positions_file="$(arg initial_positions_file)" use_sim="$(arg use_sim)" />
+    <xacro:robot_ros2_control name="robot" initial_positions_file="$(arg initial_positions_file)" use_sim="$(arg use_sim)" />
 </robot>

File: src/robot_description_moveit/config/robot.ros2_control.xacro (robot description, xacro)
@@ -1,76 +1,75 @@
 <?xml version="1.0"?>
 <robot xmlns:xacro="http://www.ros.org/wiki/xacro">
-    <xacro:macro name="robot_ros2_control" params="name initial_positions_file">
-        <xacro:property name="initial_positions" value="${xacro.load_yaml(initial_positions_file)['initial_positions']}"/>
-        <ros2_control name="${name}" type="system">
-            <hardware>
-                <!-- By default, set up controllers for simulation. This won't work on real hardware -->
-                <plugin>mock_components/GenericSystem</plugin>
-            </hardware>
-            <joint name="joint_1">
-                <command_interface name="position"/>
-                <command_interface name="velocity"/>
-                <state_interface name="position">
-                  <param name="initial_value">${initial_positions['joint_1']}</param>
-                </state_interface>
-                <state_interface name="velocity"/>
-            </joint>
-            <joint name="joint_2">
-                <command_interface name="position"/>
-                <command_interface name="velocity"/>
-                <state_interface name="position">
-                  <param name="initial_value">${initial_positions['joint_2']}</param>
-                </state_interface>
-                <state_interface name="velocity"/>
-            </joint>
-            <joint name="joint_3">
-                <command_interface name="position"/>
-                <command_interface name="velocity"/>
-                <state_interface name="position">
-                  <param name="initial_value">${initial_positions['joint_3']}</param>
-                </state_interface>
-                <state_interface name="velocity"/>
-            </joint>
-            <joint name="joint_4">
-                <command_interface name="position"/>
-                <command_interface name="velocity"/>
-                <state_interface name="position">
-                  <param name="initial_value">${initial_positions['joint_4']}</param>
-                </state_interface>
-                <state_interface name="velocity"/>
-            </joint>
-            <joint name="joint_5">
-                <command_interface name="position"/>
-                <command_interface name="velocity"/>
-                <state_interface name="position">
-                  <param name="initial_value">${initial_positions['joint_5']}</param>
-                </state_interface>
-                <state_interface name="velocity"/>
-            </joint>
-            <joint name="joint_6">
-                <command_interface name="position"/>
-                <command_interface name="velocity"/>
-                <state_interface name="position">
-                  <param name="initial_value">${initial_positions['joint_6']}</param>
-                </state_interface>
-                <state_interface name="velocity"/>
-            </joint>
-            <joint name="joint_gl">
-                <command_interface name="position"/>
-                <command_interface name="velocity"/>
-                <state_interface name="position">
-                  <param name="initial_value">${initial_positions['joint_gl']}</param>
-                </state_interface>
-                <state_interface name="velocity"/>
-            </joint>
-            <joint name="joint_gr">
-                <command_interface name="position"/>
-                <command_interface name="velocity"/>
-                <state_interface name="position">
-                  <param name="initial_value">${initial_positions['joint_gr']}</param>
-                </state_interface>
-                <state_interface name="velocity"/>
-            </joint>
-        </ros2_control>
-    </xacro:macro>
+  <!-- Macro defining ros2_control block -->
+  <xacro:macro name="robot_ros2_control"
+               params="name:='robot_system'
+                       initial_positions_file:=''
+                       use_sim:='false'">
+    <!-- Load initial joint positions if a file is provided -->
+    <xacro:if value="${initial_positions_file != ''}">
+      <xacro:property
+        name="initial_positions"
+        value="${xacro.load_yaml(initial_positions_file)['initial_positions']}" />
+    </xacro:if>
+    <ros2_control name="${name}" type="system">
+      <hardware>
+        <xacro:if value="${use_sim}">
+          <plugin>gz_ros2_control/GazeboSimSystem</plugin>
+        </xacro:if>
+        <xacro:unless value="${use_sim}">
+          <plugin>mock_components/GenericSystem</plugin>
+          <param name="calculate_dynamics">true</param>
+        </xacro:unless>
+      </hardware>
+      <!-- Joints -->
+      <joint name="joint_1">
+        <command_interface name="position"/>
+        <state_interface name="position"/>
+        <command_interface name="velocity"/>
+        <state_interface name="velocity"/>
+      </joint>
+      <joint name="joint_2">
+        <command_interface name="position"/>
+        <state_interface name="position"/>
+        <command_interface name="velocity"/>
+        <state_interface name="velocity"/>
+      </joint>
+      <joint name="joint_3">
+        <command_interface name="position"/>
+        <state_interface name="position"/>
+        <command_interface name="velocity"/>
+        <state_interface name="velocity"/>
+      </joint>
+      <joint name="joint_4">
+        <command_interface name="position"/>
+        <state_interface name="position"/>
+        <command_interface name="velocity"/>
+        <state_interface name="velocity"/>
+      </joint>
+      <joint name="joint_5">
+        <command_interface name="position"/>
+        <state_interface name="position"/>
+        <command_interface name="velocity"/>
+        <state_interface name="velocity"/>
+      </joint>
+      <joint name="joint_6">
+        <command_interface name="position"/>
+        <state_interface name="position"/>
+        <command_interface name="velocity"/>
+        <state_interface name="velocity"/>
+      </joint>
+      <joint name="joint_gl">
+        <command_interface name="position"/>
+        <state_interface name="position"/>
+        <command_interface name="velocity"/>
+        <state_interface name="velocity"/>
+      </joint>
+      <joint name="joint_gr">
+        <command_interface name="position"/>
+        <state_interface name="position"/>
+        <command_interface name="velocity"/>
+        <state_interface name="velocity"/>
+      </joint>
+    </ros2_control>
+  </xacro:macro>
 </robot>

Commit message: Camera Link

File: src/robot_description/urdf/gazebo.xacro (robot description, xacro)
@@ -11,5 +11,5 @@
         <visual>
             <geometry>
-                <box size="0.05 0.05 0.05"/>
+                <mesh filename="package://robot_description/meshes/astra_cam.stl" />
             </geometry>
             <material name="black">
@@ -19,12 +19,12 @@
         <collision>
             <geometry>
-                 <box size="0.05 0.05 0.05"/>
+                <mesh filename="package://robot_description/meshes/astra_cam.stl" />
             </geometry>
         </collision>
     </link>
     <joint name="camera_joint" type="fixed">
-        <parent link="base_link"/>
+        <parent link="world"/>
         <child link="camera_link"/>
-        <origin xyz="0.5 0 0.5" rpy="0 0 0"/>
+        <origin xyz="0.8 0 2" rpy="3.1416 0 1.5707"/>
     </joint>
 </robot>

File: src/robot_description/urdf/robot.xacro (robot description, xacro)
@@ -179,5 +179,5 @@
     <axis xyz="0 0 1" />
     <limit
-      lower="-3.1415" upper="3.1415"
+      lower="-1.5707" upper="1.5707"
       effort="1000" velocity="5.0" />
   </joint>
@@ -252,5 +252,5 @@
     <axis xyz="0 0 1" />
     <limit
-      lower="-3.1415" upper="3.1415"
+      lower="-1.5707" upper="1.5707"
       effort="1000" velocity="5.0" />
   </joint>
@@ -289,5 +289,5 @@
     <axis xyz="1 0 0" />
     <limit
-      lower="0" upper="0.1"
+      lower="0" upper="0.02"
       effort="50" velocity="0.05" />
   </joint>
@@ -325,5 +325,5 @@
     <axis xyz="1 0 0" />
     <limit
-      lower="0" upper="0.1"
+      lower="0" upper="0.02"
       effort="50" velocity="0.05" />
   </joint>

Commit message: Update PKG

File: src/robot_description/urdf/gazebo.xacro (robot description, xacro)
@@ -3,6 +3,10 @@
     <xacro:if value="$(arg use_sim)">
         <gazebo>
-            <plugin filename="libgz_ros2_control-system.so" name="gz_ros2_control::GazeboSimROS2ControlPlugin">
-                <parameters>$(find robot_moveit)/config/ros2_controllers.yaml</parameters>
+            <plugin
+                filename="libgz_ros2_control-system.so"
+                name="gz_ros2_control::GazeboSimROS2ControlPlugin">
+                <parameters>
+                    $(find robot_control)/config/robot_controllers.yaml
+                </parameters>
             </plugin>
         </gazebo>

File: src/robot_description/urdf/robot.urdf.xacro (robot description, xacro)
@@ -1,18 +1,18 @@
 <?xml version="1.0"?>
 <robot xmlns:xacro ="http://www.ros.org/wiki/xacro" name="robot">
-    <xacro:arg name ="use_sim"
-            default ="true" />
+    <xacro:arg name ="use_sim" default ="true" />
+    <xacro:arg name ="use_mock_hardware" default ="false" />
     <xacro:arg name ="initial_positions_file"
-            default ="$(find robot_moveit)/config/initial_positions.yaml" />
-    <xacro:include filename =   "$(find robot_description)/urdf/materials.xacro" />
-    <xacro:include filename =   "$(find robot_description)/urdf/robot.xacro" />
-    <xacro:include filename =   "$(find robot_description)/urdf/sensors.xacro"/>
-    <xacro:include filename =   "$(find robot_description)/urdf/ros2_control.xacro" />
-    <xacro:include filename =   "$(find robot_description)/urdf/gazebo.xacro" />
+            default ="$(find robot_control)/config/initial_positions.yaml" />
+    <xacro:include filename ="$(find robot_description)/urdf/materials.xacro" />
+    <xacro:include filename ="$(find robot_description)/urdf/robot.xacro" />
+    <xacro:include filename ="$(find robot_description)/urdf/sensors.xacro"/>
+    <xacro:include filename ="$(find robot_description)/urdf/ros2_control.xacro" />
+    <xacro:include filename ="$(find robot_description)/urdf/gazebo.xacro" />
     <xacro:base_camera
-            parent_link             ="base_link"
-            base_link               ="astra_link"
-            camera_name             ="astra_depth"
-            frame_name              ="astra_link"/>
+            parent_link     ="base_link"
+            base_link       ="astra_link"
+            camera_name     ="astra_depth"
+            frame_name      ="astra_link"/>
     <xacro:robot_ros2_control
             name                    ="robot"

File: src/robot_description/urdf/robot.xacro (robot description, xacro)
@@ -334,22 +334,22 @@
   </joint>
   <gazebo reference="gripper_l">
-    <mu1>1000.0</mu1>
-    <mu2>1000.0</mu2>
-    <kp>1000000.0</kp>
-    <kd>1.0</kd>
-    <minDepth>0.001</minDepth>
-    <maxVel>0.1</maxVel>
-    <selfCollide>false</selfCollide>
-    <material>Gazebo/Grey</material>
+    <mu1>         1000.0</mu1>
+    <mu2>         1000.0</mu2>
+    <kp>          1000000.0</kp>
+    <kd>          1.0</kd>
+    <minDepth>    0.001</minDepth>
+    <maxVel>      0.1</maxVel>
+    <selfCollide> false</selfCollide>
+    <material>    Gazebo/Grey</material>
   </gazebo>
   <gazebo reference="gripper_r">
-    <mu1>1000.0</mu1>
-    <mu2>1000.0</mu2>
-    <kp>1000000.0</kp>
-    <kd>1.0</kd>
-    <minDepth>0.001</minDepth>
-    <maxVel>0.1</maxVel>
-    <selfCollide>false</selfCollide>
-    <material>Gazebo/Grey</material>
+    <mu1>         1000.0</mu1>
+    <mu2>         1000.0</mu2>
+    <kp>          1000000.0</kp>
+    <kd>          1.0</kd>
+    <minDepth>    0.001</minDepth>
+    <maxVel>      0.1</maxVel>
+    <selfCollide> false</selfCollide>
+    <material>    Gazebo/Grey</material>
   </gazebo>
 </robot>

File: src/robot_description/urdf/ros2_control.xacro (robot description, xacro)
@@ -3,26 +3,31 @@
   <!-- Macro defining ros2_control block -->
   <xacro:macro name   ="robot_ros2_control"
-               params ="name:='robot_system'
-                       initial_positions_file:=''
-                       use_sim:='false'">
+               params =
+                      "name                   :='robot_system'
+                       initial_positions_file :=''
+                       use_sim                :='false'
+                       use_mock               :='true' ">
     <!-- Load initial joint positions if a file is provided -->
-    <xacro:if value="${initial_positions_file != ''}">
+    <xacro:if value ="${initial_positions_file != ''}">
       <xacro:property
-        name="initial_positions"
-        value="${xacro.load_yaml(initial_positions_file)['initial_positions']}" />
+              name  ="initial_positions"
+              value ="${xacro.load_yaml(initial_positions_file)['initial_positions']}" />
     </xacro:if>
     <ros2_control name="${name}" type="system">
       <hardware>
+        <!-- SIM (Gazebo) -->
         <xacro:if value="${use_sim}">
           <plugin>gz_ros2_control/GazeboSimSystem</plugin>
         </xacro:if>
+        <!-- REAL  -->
         <xacro:unless value="${use_sim}">
-          <!--_____________ Plugin hardware cũ ______________-->
-          <plugin>mock_components/GenericSystem</plugin>
-          <param name="calculate_dynamics">true</param>
-          <!--_____________ Plugin hardware mới ______________-->
-          <!--plugin>robot_hardware/RobotSystemHardware</plugin>
-          <param name="port">${port}</param>
-          <param name="baud">${baud}</param-->
+          <!-- MOCK HARDWARE -->
+          <xacro:if value="${use_mock}">
+            <plugin>mock_components/GenericSystem</plugin>
+          </xacro:if>
+          <!-- REAL HARDWARE -->
+          <xacro:unless value="${use_mock}">
+            <plugin>robot_hardware_interface/RobotSystemHardware</plugin>
+          </xacro:unless>
         </xacro:unless>
       </hardware>

File: src/robot_description/urdf/sensors.xacro (robot description, xacro)
@@ -25,5 +25,4 @@
     </link>
     <link           name  ="${base_link}_optical"/>
-    <!-- chỉnh lại pose camera tại đây -->
     <joint          name  ="${base_link}_joint"         type  ="fixed">
       <parent       link  ="${parent_link}"/>
@@ -31,5 +30,4 @@
       <origin       xyz   ="0.6 0 1.0" rpy="${pi} 0 ${pi/2}"/>
     </joint>
-    <!-- Chỉnh lại optical frame -->
     <joint          name  ="${base_link}_optical_joint" type  ="fixed">
       <parent       link  ="${base_link}"/>
@@ -44,5 +42,4 @@
         <visualize>true</visualize>
         <topic>astra/rgb/image_raw</topic>
-        <gz_frame_id>${base_link}_optical</gz_frame_id>
         <camera>
           <image>
@@ -65,5 +62,4 @@
         <visualize>true</visualize>
         <topic>astra/depth/image_raw</topic>
-        <gz_frame_id>${base_link}_optical</gz_frame_id>
         <camera>
           <image>
