Commit message: camera

File: src/robot_description/urdf/robot.xacro (robot description, xacro)
@@ -251,85 +251,85 @@
   <!-- ________________ DEFINE JOINT ________________________________________________________________________ -->
   <!-- World-Base Joint -->
-  <joint    name  ="virtual_joint"    type      ="fixed">
-    <origin xyz   ="0 0 0"            rpy       ="0 0 0"/>
+  <joint    name  ="virtual_joint"         type      ="fixed">
+    <origin xyz   ="0 0 0"                 rpy       ="0 0 0"/>
     <parent link  ="world"/>
     <child  link  ="base_link"/>
   </joint>
-  <joint    name  ="tcp_joint"        type      ="fixed">
-    <origin xyz   ="0 0 0.08"         rpy       ="0 0 0"/>
+  <joint    name  ="tcp_joint"             type      ="fixed">
+    <origin xyz   ="0 0 0.08"              rpy       ="0 0 0"/>
     <parent link  ="link_6"/>
     <child  link  ="tcp_link"/>
   </joint>
   <!-- JOINT 1 -->
-  <joint    name  ="joint_1"          type      ="revolute">
-    <origin xyz   ="0 0 0.01"         rpy       ="0 0 0" />
+  <joint    name  ="joint_1"               type      ="revolute">
+    <origin xyz   ="0 0 0.01"              rpy       ="0 0 0" />
     <parent link  ="base_link" />
     <child  link  ="link_1" />
     <axis   xyz   ="0 0 1" />
-    <limit  lower ="-2.0943"          upper     ="2.0943"
-            effort="1000"             velocity  ="5.0" />
+    <limit  lower ="-2.0943"               upper     ="2.0943"
+            effort="1000"                  velocity  ="5.0" />
   </joint>
   <!-- JOINT 2 -->
-  <joint    name  ="joint_2"          type      ="revolute">
-    <origin xyz   ="0.1 0.05 0.24313" rpy       ="${-pi/2} ${-pi/2} 0" />
+  <joint    name  ="joint_2"               type      ="revolute">
+    <origin xyz   ="0.1 0.05 0.24313"      rpy       ="${-pi/2} ${-pi/2} 0" />
     <parent link  ="link_1" />
     <child  link  ="link_2" />
     <axis   xyz   ="0 0 1" />
-    <limit  lower ="-1.5707"          upper     ="2.6179"
-            effort="1000"             velocity  ="5.0" />
+    <limit  lower ="-1.5707"               upper     ="2.6179"
+            effort="1000"                  velocity  ="5.0" />
   </joint>
   <!-- JOINT 3 -->
-  <joint    name  ="joint_3"          type      ="revolute">
-    <origin xyz   ="0.25 0 -0.01"     rpy       ="0 0 ${pi/2}" />
+  <joint    name  ="joint_3"               type      ="revolute">
+    <origin xyz   ="0.25 0 -0.01"          rpy       ="0 0 ${pi/2}" />
     <parent link  ="link_2" />
     <child  link  ="link_3" />
     <axis   xyz   ="0 0 1" />
-    <limit  lower ="-1.5707"          upper     ="1.5707"
-            effort="1000"             velocity  ="5.0" />
+    <limit  lower ="-1.5707"               upper     ="1.5707"
+            effort="1000"                  velocity  ="5.0" />
   </joint>
   <!-- JOINT 4 -->
-  <joint    name  ="joint_4"            type    ="revolute">
-    <origin xyz   ="0.103 -0.09 -0.04"  rpy     ="0 ${pi/2} 0" />
+  <joint    name  ="joint_4"               type    ="revolute">
+    <origin xyz   ="0.103 -0.09 -0.04"     rpy     ="0 ${pi/2} 0" />
     <parent link  ="link_3" />
     <child  link  ="link_4" />
     <axis   xyz   ="0 0 1" />
-    <limit  lower ="-1.5707"          upper     ="1.5707"
-            effort="1000"             velocity  ="5.0" />
+    <limit  lower ="-1.5707"               upper     ="1.5707"
+            effort="1000"                  velocity  ="5.0" />
   </joint>
   <!-- JOINT 5 -->
-  <joint    name  ="joint_5"            type    ="revolute">
-    <origin xyz   ="-0.0134 0 0.12"     rpy     ="${pi} ${-pi/2} ${pi}" />
+  <joint    name  ="joint_5"               type    ="revolute">
+    <origin xyz   ="-0.0134 0 0.12"        rpy     ="${pi} ${-pi/2} ${pi}" />
     <parent link  ="link_4" />
     <child  link  ="link_5" />
     <axis   xyz   ="0 0 1" />
-    <limit  lower ="-1.5707"          upper    ="1.5707"
-            effort="1000"             velocity ="5.0" />
+    <limit  lower ="-1.5707"               upper    ="1.5707"
+            effort="1000"                  velocity ="5.0" />
   </joint>
   <!-- JOINT 6 -->
-  <joint    name  ="joint_6"          type    ="revolute">
-    <origin xyz   ="0.136 0 -0.01483" rpy     ="0 ${-pi/2} ${pi}" />
+  <joint    name  ="joint_6"               type    ="revolute">
+    <origin xyz   ="0.136 0 -0.01483"      rpy     ="0 ${-pi/2} ${pi}" />
     <parent link  ="link_5" />
     <child  link  ="link_6" />
     <axis   xyz   ="0 0 1" />
-    <limit  lower ="-1.5707"          upper     ="1.5707"
-            effort="1000"             velocity  ="5.0" />
+    <limit  lower ="-1.5707"               upper     ="1.5707"
+            effort="1000"                  velocity  ="5.0" />
   </joint>
   <!-- joint_gl -->
-  <joint    name  ="joint_gl"         type      ="prismatic">
-    <origin xyz   ="0.0021 0 0.0668"  rpy       ="0 0 0" />
+  <joint    name  ="joint_gl"              type      ="prismatic">
+    <origin xyz   ="0.0021 0 0.0668"       rpy       ="0 0 0" />
     <parent link  ="link_6" />
     <child  link  ="gripper_l" />
     <axis   xyz   ="1 0 0" />
-    <limit  lower ="0"                upper     ="0.02"
-            effort="50"               velocity  ="0.05" />
+    <limit  lower ="-0.001"                upper     ="0.02"
+            effort="50"                    velocity  ="0.05" />
   </joint>
   <!-- joint_gr -->
-  <joint    name  ="joint_gr"         type      ="prismatic">
-    <origin xyz   ="-0.0021 0 0.0668" rpy       ="0 0 ${pi}" />
+  <joint    name  ="joint_gr"              type      ="prismatic">
+    <origin xyz   ="-0.0021 0 0.0668"      rpy       ="0 0 ${pi}" />
     <parent link  ="link_6" />
     <child  link  ="gripper_r" />
     <axis   xyz   ="1 0 0" />
-    <limit  lower ="0"                upper     ="0.02"
-            effort="50"               velocity  ="0.05" />
+    <limit  lower ="-0.001"                upper     ="0.02"
+            effort="50"                    velocity  ="0.05" />
   </joint>
   <gazebo reference="gripper_l">

File: src/robot_description/urdf/sensors.xacro (robot description, xacro)
@@ -37,8 +37,12 @@
       <origin       xyz   ="0 0 0" rpy="0 0 0"/>
     </joint>
-    <!--gazebo reference="camera_link">
-      <sensor name="camera" type="camera">
+    <gazebo reference="${base_link}">
+      <sensor name="astra_rgb" type="camera">
+        <always_on>true</always_on>
+        <update_rate>30</update_rate>
+        <visualize>true</visualize>
+        <topic>astra/rgb/image_raw</topic>
+        <gz_frame_id>${base_link}_optical</gz_frame_id>
         <camera>
-          <horizontal_fov>1.3962634</horizontal_fov>
           <image>
             <width>640</width>
@@ -47,21 +51,29 @@
           </image>
           <clip>
-            <near>0.1</near>
-            <far>15</far>
+            <near>0.05</near>
+            <far>8.0</far>
           </clip>
-          <noise>
-            <type>gaussian</type>
-            <mean>0.0</mean>
-            <stddev>0.007</stddev>
-          </noise>
-          <optical_frame_id>camera_link_optical</optical_frame_id>
-          <camera_info_topic>camera/camera_info</camera_info_topic>
         </camera>
-        <always_on>1</always_on>
-        <update_rate>20</update_rate>
-        <visualize>true</visualize>
-        <topic>camera/image</topic>
       </sensor>
-    </gazebo-->
+    </gazebo>
+    <gazebo reference="${base_link}">
+      <sensor name="astra_depth" type="depth">
+        <always_on>true</always_on>
+        <update_rate>30</update_rate>
+        <visualize>false</visualize>
+        <topic>astra/depth/image_raw</topic>
+        <gz_frame_id>${base_link}_optical</gz_frame_id>
+        <camera>
+          <image>
+            <width>640</width>
+            <height>480</height>
+          </image>
+          <clip>
+            <near>0.05</near>
+            <far>8.0</far>
+          </clip>
+        </camera>
+      </sensor>
+    </gazebo>
   </xacro:macro>
 </robot>

Commit message: fix Hardware interface, fix cmd control vel, add pkg robot_task_manager

File: src/robot_description/urdf/robot.xacro (robot description, xacro)
@@ -263,5 +263,5 @@
   <!-- JOINT 1 -->
   <joint    name  ="joint_1"               type      ="revolute">
-    <origin xyz   ="0 0 0.01"              rpy       ="0 0 0" />
+    <origin xyz   ="0 0 0.05"              rpy       ="0 0 0" />
     <parent link  ="base_link" />
     <child  link  ="link_1" />
@@ -272,5 +272,5 @@
   <!-- JOINT 2 -->
   <joint    name  ="joint_2"               type      ="revolute">
-    <origin xyz   ="0.1 0.05 0.24313"      rpy       ="${-pi/2} ${-pi/2} 0" />
+    <origin xyz   ="0.1 0.04 0.24313"      rpy       ="${-pi/2} ${-pi/2} 0" />
     <parent link  ="link_1" />
     <child  link  ="link_2" />
@@ -281,5 +281,5 @@
   <!-- JOINT 3 -->
   <joint    name  ="joint_3"               type      ="revolute">
-    <origin xyz   ="0.25 0 -0.01"          rpy       ="0 0 ${pi/2}" />
+    <origin xyz   ="0.25 0 0.0"          rpy       ="0 0 ${pi/2}" />
     <parent link  ="link_2" />
     <child  link  ="link_3" />
@@ -299,5 +299,5 @@
   <!-- JOINT 5 -->
   <joint    name  ="joint_5"               type    ="revolute">
-    <origin xyz   ="-0.0134 0 0.12"        rpy     ="${pi} ${-pi/2} ${pi}" />
+    <origin xyz   ="-0.05 0 0.12"        rpy     ="${pi} ${-pi/2} ${pi}" />
     <parent link  ="link_4" />
     <child  link  ="link_5" />
@@ -308,5 +308,5 @@
   <!-- JOINT 6 -->
   <joint    name  ="joint_6"               type    ="revolute">
-    <origin xyz   ="0.136 0 -0.01483"      rpy     ="0 ${-pi/2} ${pi}" />
+    <origin xyz   ="0.132 0 -0.05"      rpy     ="0 ${-pi/2} ${pi}" />
     <parent link  ="link_5" />
     <child  link  ="link_6" />

File: src/robot_description/urdf/ros2_control.xacro (robot description, xacro)
@@ -7,6 +7,6 @@
                        initial_positions_file :=''
                        use_sim                :='false'
-                       use_mock               :='true' ">
-    <!-- Load initial joint positions if a file is provided -->
+                       use_mock               :='false' ">
+    <!-- Load initial joint positions if a file is provided true -->
     <xacro:if value ="${initial_positions_file != ''}">
       <xacro:property
