Commit message: Commit 24060

File: src/robot_description/urdf/robot.urdf.xacro (robot description, xacro)
@@ -12,10 +12,11 @@
     <xacro:base_camera
             parent_link     ="base_link"
-            base_link       ="astra_link"
+            base_link       ="astra_base"
             camera_name     ="astra_depth"
-            frame_name      ="astra_link"/>
+            frame_name      ="astra"/>
     <xacro:robot_ros2_control
             name                    ="robot"
             initial_positions_file  ="$(arg initial_positions_file)"
-            use_sim                 ="$(arg use_sim)" />
+            use_sim                 ="$(arg use_sim)"
+            use_mock                ="$(arg use_mock_hardware)" />
 </robot>

File: src/robot_description/urdf/robot.xacro (robot description, xacro)
@@ -28,5 +28,5 @@
       <origin xyz ="0 0 0" rpy ="0 0 0" />
       <geometry>
-        <mesh filename  ="package://robot_description/meshes/base_link.stl" />
+        <mesh filename  ="package://robot_description/meshes/dae/base_link.dae" />
       </geometry>
     </collision>
@@ -53,7 +53,7 @@
     </visual>
     <collision>
-      <origin xyz ="0 0 0" rpy  ="0 0 0" />
-      <geometry>
-        <mesh filename  ="package://robot_description/meshes/link_1.stl" />
+      <origin xyz ="0 0 0" rpy ="0 0 0" />
+      <geometry>
+        <mesh filename  ="package://robot_description/meshes/dae/link_1.dae" />
       </geometry>
     </collision>
@@ -80,7 +80,7 @@
     </visual>
     <collision>
-      <origin xyz="0 0 0" rpy="0 0 0" />
-      <geometry>
-        <mesh filename="package://robot_description/meshes/link_2.stl" />
+      <origin xyz ="0 0 0" rpy ="0 0 0" />
+      <geometry>
+        <mesh filename  ="package://robot_description/meshes/dae/link_2.dae" />
       </geometry>
     </collision>
@@ -107,7 +107,7 @@
     </visual>
     <collision>
-      <origin  xyz="0 0 0" rpy="0 0 0" />
-      <geometry>
-        <mesh  filename="package://robot_description/meshes/link_3.stl" />
+      <origin xyz ="0 0 0" rpy ="0 0 0" />
+      <geometry>
+        <mesh filename  ="package://robot_description/meshes/dae/link_3.dae" />
       </geometry>
     </collision>
@@ -134,7 +134,7 @@
     </visual>
     <collision>
-      <origin  xyz="0 0 0"  rpy="0 0 0" />
-      <geometry>
-        <mesh filename="package://robot_description/meshes/link_4.stl" />
+      <origin xyz ="0 0 0" rpy ="0 0 0" />
+      <geometry>
+        <mesh filename  ="package://robot_description/meshes/dae/link_4.dae" />
       </geometry>
     </collision>
@@ -161,7 +161,7 @@
     </visual>
     <collision>
-      <origin  xyz="0 0 0"  rpy="0 0 0" />
-      <geometry>
-        <mesh filename  ="package://robot_description/meshes/link_5.stl" />
+      <origin xyz ="0 0 0" rpy ="0 0 0" />
+      <geometry>
+        <mesh filename  ="package://robot_description/meshes/dae/link_5.dae" />
       </geometry>
     </collision>
@@ -188,7 +188,7 @@
     </visual>
     <collision>
-      <origin  xyz  ="0 0 0"  rpy ="0 0 0" />
-      <geometry>
-        <mesh filename  ="package://robot_description/meshes/link_6.stl" />
+      <origin xyz ="0 0 0" rpy ="0 0 0" />
+      <geometry>
+        <mesh filename  ="package://robot_description/meshes/dae/link_6.dae" />
       </geometry>
     </collision>
@@ -216,7 +216,7 @@
     </visual>
     <collision>
-      <origin xyz="0 0 0" rpy="0 0 0" />
-      <geometry>
-        <mesh filename  ="package://robot_description/meshes/gripper_l.stl" />
+      <origin xyz ="0 0 0" rpy ="0 0 0" />
+      <geometry>
+        <mesh filename  ="package://robot_description/meshes/dae/gripper_l.dae" />
       </geometry>
     </collision>
@@ -243,7 +243,7 @@
     </visual>
     <collision>
-      <origin xyz ="0 0 0" rpy  ="0 0 0" />
-      <geometry>
-        <mesh  filename ="package://robot_description/meshes/gripper_r.stl" />
+      <origin xyz ="0 0 0" rpy ="0 0 0" />
+      <geometry>
+        <mesh filename  ="package://robot_description/meshes/dae/gripper_r.dae" />
       </geometry>
     </collision>

File: src/robot_description/urdf/sensors.xacro (robot description, xacro)
@@ -24,22 +24,23 @@
       </collision>
     </link>
-    <link           name  ="${base_link}_optical"/>
+    <link           name  ="${frame_name}_optical"/>
     <joint          name  ="${base_link}_joint"         type  ="fixed">
       <parent       link  ="${parent_link}"/>
       <child        link  ="${base_link}"/>
-      <origin       xyz   ="0.6 0 1.0" rpy="${pi} 0 ${pi/2}"/>
+      <origin       xyz   ="0.7 0 0.9" rpy="${pi} ${pi/12} 0"/>
     </joint>
+    <!-- rpy= ${pi} ${pi/12} 0-->
     <joint          name  ="${base_link}_optical_joint" type  ="fixed">
       <parent       link  ="${base_link}"/>
-      <child        link  ="${base_link}_optical"/>
+      <child        link  ="${frame_name}_optical"/>
       <origin       xyz   ="0 0 0" rpy="0 0 0"/>
     </joint>
-    <gazebo reference="${base_link}">
+    <gazebo reference="${frame_name}_optical">
       <sensor name="astra_rgb" type="camera">
-        <pose>0 0 0 0 ${-pi/2} 0</pose>
+        <pose>0 0 0  0  ${-pi/2} ${pi/2}  </pose>
         <always_on>true</always_on>
-        <update_rate>30</update_rate>
+        <update_rate>20</update_rate>
         <visualize>true</visualize>
-        <topic>astra/rgb/image_raw</topic>
+        <topic>astra_sim/rgb/image_raw</topic>
         <camera>
           <image>
@@ -55,11 +56,11 @@
       </sensor>
     </gazebo>
-    <gazebo reference="${base_link}">
+    <gazebo reference="${frame_name}_optical">
       <sensor name="astra_depth" type="depth">
-        <pose>0 0 0 0 ${-pi/2} 0</pose>
+        <pose>0 0 0  0  ${-pi/2} ${pi/2}  </pose>
         <always_on>true</always_on>
-        <update_rate>30</update_rate>
+        <update_rate>20</update_rate>
         <visualize>true</visualize>
-        <topic>astra/depth/image_raw</topic>
+        <topic>astra_sim/depth/image_raw</topic>
         <camera>
           <image>
